File: schema-pcb/treuil-handi.sch (KiCad schematic (older format))
At the start: 5 parts, among them K1 PPM, SW1 calibration, U2 AS5048B Pot, U3 AS5048B moteur

Commit message: ajout R pull ups i2c + photo proto
Parts:
- added R1, R2: 470, ~, symbol R
Connections:
- net 3V3: now also R1.1, R2.1
- net at SHIELD1.20 (SDA), U2.1 (SDA/CS), U3.1 (SDA/CS): now also R1.2
- net at SHIELD1.21 (SCL), U2.2 (SCL/SCK), U3.2 (SCL/SCK): now also R2.2
Changed lines of the file:
@@
-EESchema Schematic File Version 2  date 30/06/2014 12:20:45
+EESchema Schematic File Version 2  date 02/07/2014 22:55:28
 LIBS:power
 LIBS:device
@@
 Sheet 1 1
 Title ""
-Date "30 jun 2014"
+Date "2 jul 2014"
 Rev ""
 Comp ""
@@
 Wire Wire Line
 	4900 1600 4900 1900
+$Comp
+L R R1
+U 1 1 53B47095
+P 4600 3350
+F 0 "R1" V 4680 3350 40  0000 C CNN
+F 1 "470" V 4607 3351 40  0000 C CNN
+F 2 "~" V 4530 3350 30  0000 C CNN
+F 3 "~" H 4600 3350 30  0000 C CNN
+	1    4600 3350
+	1    0    0    -1
+$EndComp
+$Comp
+L R R2
+U 1 1 53B470A4
+P 4850 3350
+F 0 "R2" V 4930 3350 40  0000 C CNN
+F 1 "470" V 4857 3351 40  0000 C CNN
+F 2 "~" V 4780 3350 30  0000 C CNN
+F 3 "~" H 4850 3350 30  0000 C CNN
+	1    4850 3350
+	1    0    0    -1
+$EndComp
+$Comp
+L 3V3 #PWR?
+U 1 1 53B470D1
+P 4700 3000
+F 0 "#PWR?" H 4700 3100 40  0001 C CNN
+F 1 "3V3" H 4700 3125 40  0000 C CNN
+F 2 "" H 4700 3000 60  0000 C CNN
+F 3 "" H 4700 3000 60  0000 C CNN
+	1    4700 3000
+	1    0    0    -1
+$EndComp
+Wire Wire Line
+	4600 3600 4600 3700
+Connection ~ 4600 3700
+Wire Wire Line
+	4850 3600 4850 3800
+Connection ~ 4850 3800
+Wire Wire Line
+	4600 3000 4850 3000
+Wire Wire Line
+	4600 3000 4600 3100
+Wire Wire Line
+	4850 3000 4850 3100
+Connection ~ 4700 3000
 $EndSCHEMATC
